Commit message: flatでの検証

File: urdf/vehicle_4ws_real.xacro (robot description, xacro)
@@ -17,9 +17,9 @@
 <xacro:property name="front_steering_friction" value="${front_steering_mu * gravitational_acceleration * 0.25*vehicle_body_mass}" />
 <!-- rearは駆動輪なので、入力以外で動かないように設定 -->
-<xacro:property name="wheel_joint_damping" value="5.0"/>
-<xacro:property name="wheel_joint_mu" value="0.1" />
+<xacro:property name="wheel_joint_damping" value="0.2"/>
+<xacro:property name="wheel_joint_mu" value="0.05" />
 <xacro:property name="wheel_joint_friction" value="${wheel_joint_mu* gravitational_acceleration * wheel_mass }" />
 <xacro:property name="steering_damping" value="20.0" />
-<xacro:property name="steering_mu" value="0.5" />
+<xacro:property name="steering_mu" value="0.01" />
 <xacro:property name="steering_friction" value="${steering_mu * gravitational_acceleration * 0.25*vehicle_body_mass}" />
 <!-- rotationは共通 -->

Commit message: 後輪をeffortに変更

File: urdf/vehicle_4ws_real.xacro (robot description, xacro)
@@ -272,5 +272,5 @@
   <dynamics damping="${front_steering_damping}" friction="${front_steering_friction}"/>
   <axis xyz="0.0 0.0 1.0"/>
-  <limit upper="1.5708" lower="-1.5708" effort="100" velocity="100"/>
+  <limit upper="1.047" lower="-1.047" effort="100" velocity="100"/>
 </joint>
 <joint name="front_right_wheel" type="continuous">
@@ -295,5 +295,5 @@
   <dynamics damping="${front_steering_damping}" friction="${front_steering_friction}"/>
   <axis xyz="0.0 0.0 1.0"/>
-  <limit upper="1.5708" lower="-1.5708" effort="100" velocity="100"/>
+  <limit upper="1.047" lower="-1.047" effort="100" velocity="100"/>
 </joint>
 <joint name="front_left_wheel" type="continuous">

Commit message: URDFの接地面の摩擦を変更

File: urdf/vehicle_4ws_real.xacro (robot description, xacro)
@@ -23,4 +23,11 @@
 <xacro:property name="steering_mu" value="0.01" />
 <xacro:property name="steering_friction" value="${steering_mu * gravitational_acceleration * 0.25*vehicle_body_mass}" />
+<!-- wheelの接地面の摩擦などを定義 -->
+<xacro:property name="wheel_surface_mu1" value="5.0"/>
+<xacro:property name="wheel_surface_mu2" value="5.0" />
+<xacro:property name="wheel_kp" value="1e5" />
+<xacro:property name="wheel_kd" value="1.0" />
+<xacro:property name="wheel_minDepth" value="0.01" />
+<xacro:property name="wheel_maxVel" value="0.1" />
 <!-- rotationは共通 -->
 <xacro:property name="rotational_joint_damping" value="0.01" />
@@ -111,4 +118,65 @@
   </collision>
 </link>
+<link name="new_hinge_3">
+  <inertial>
+    <origin xyz="-6.714468377522209e-05 2.5406917258941064e-07 -0.11523004751915977" rpy="0 0 0"/>
+    <mass value="4.884144703315957"/>
+    <inertia ixx="0.039519" iyy="0.032652" izz="0.021551" ixy="-0.0" iyz="0.0" ixz="-3e-05"/>
+  </inertial>
+  <visual>
+    <origin xyz="-0.45045 -0.45752 -0.356" rpy="0 0 0"/>
+    <geometry>
+      <mesh filename="package://vehicle_4ws_description/meshes/new_hinge_3.stl" scale="0.001 0.001 0.001"/>
+    </geometry>
+    <material name="_"/>
+  </visual>
+  <collision>
+    <origin xyz="-0.45045 -0.45752 -0.356" rpy="0 0 0"/>
+    <geometry>
+      <mesh filename="package://vehicle_4ws_description/meshes/new_hinge_3.stl" scale="0.001 0.001 0.001"/>
+    </geometry>
+  </collision>
+</link>
+<link name="new_hinge_2">
+  <inertial>
+    <origin xyz="-6.714468377322369e-05 2.540692444763515e-07 -0.1152300475191588" rpy="0 0 0"/>
+    <mass value="4.884144703315957"/>
+    <inertia ixx="0.039519" iyy="0.032652" izz="0.021551" ixy="0.0" iyz="0.0" ixz="-3e-05"/>
+  </inertial>
+  <visual>
+    <origin xyz="0.44955 0.34248 -0.356" rpy="0 0 0"/>
+    <geometry>
+      <mesh filename="package://vehicle_4ws_description/meshes/new_hinge_2.stl" scale="0.001 0.001 0.001"/>
+    </geometry>
+    <material name="_"/>
+  </visual>
+  <collision>
+    <origin xyz="0.44955 0.34248 -0.356" rpy="0 0 0"/>
+    <geometry>
+      <mesh filename="package://vehicle_4ws_description/meshes/new_hinge_2.stl" scale="0.001 0.001 0.001"/>
+    </geometry>
+  </collision>
+</link>
+<link name="new_hinge_4">
+  <inertial>
+    <origin xyz="-6.714468377405636e-05 2.5406924475390724e-07 -0.11523004751915963" rpy="0 0 0"/>
+    <mass value="4.884144703315957"/>
+    <inertia ixx="0.039519" iyy="0.032652" izz="0.021551" ixy="0.0" iyz="0.0" ixz="-3e-05"/>
+  </inertial>
+  <visual>
+    <origin xyz="0.44955 -0.45752 -0.356" rpy="0 0 0"/>
+    <geometry>
+      <mesh filename="package://vehicle_4ws_description/meshes/new_hinge_4.stl" scale="0.001 0.001 0.001"/>
+    </geometry>
+    <material name="_"/>
+  </visual>
+  <collision>
+    <origin xyz="0.44955 -0.45752 -0.356" rpy="0 0 0"/>
+    <geometry>
+      <mesh filename="package://vehicle_4ws_description/meshes/new_hinge_4.stl" scale="0.001 0.001 0.001"/>
+    </geometry>
+  </collision>
+</link>
+<!-- ホイールのリンク設定 -->
 <link name="new_wheel_1">
   <inertial>
@@ -129,4 +197,21 @@
       <mesh filename="package://vehicle_4ws_description/meshes/new_wheel_1.stl" scale="0.001 0.001 0.001"/>
     </geometry>
+    <!-- ここから SDF の surface/friction -->
+    <surface>
+      <friction>
+        <ode>
+          <mu>${wheel_surface_mu1}</mu>
+          <mu2>${wheel_surface_mu2}</mu2>
+        </ode>
+      </friction>
+      <contact>
+        <ode>
+          <kp>${wheel_kp}</kp>
+          <kd>${wheel_kd}</kd>
+          <minDepth>${wheel_minDepth}</minDepth>
+          <maxVel>${wheel_maxVel}</maxVel>
+        </ode>
+      </contact>
+    </surface>
   </collision>
 </link>
@@ -149,24 +234,21 @@
       <mesh filename="package://vehicle_4ws_description/meshes/new_wheel_2.stl" scale="0.001 0.001 0.001"/>
     </geometry>
-  </collision>
-</link>
-<link name="new_hinge_3">
-  <inertial>
-    <origin xyz="-6.714468377522209e-05 2.5406917258941064e-07 -0.11523004751915977" rpy="0 0 0"/>
-    <mass value="4.884144703315957"/>
-    <inertia ixx="0.039519" iyy="0.032652" izz="0.021551" ixy="-0.0" iyz="0.0" ixz="-3e-05"/>
-  </inertial>
-  <visual>
-    <origin xyz="-0.45045 -0.45752 -0.356" rpy="0 0 0"/>
-    <geometry>
-      <mesh filename="package://vehicle_4ws_description/meshes/new_hinge_3.stl" scale="0.001 0.001 0.001"/>
-    </geometry>
-    <material name="_"/>
-  </visual>
-  <collision>
-    <origin xyz="-0.45045 -0.45752 -0.356" rpy="0 0 0"/>
-    <geometry>
-      <mesh filename="package://vehicle_4ws_description/meshes/new_hinge_3.stl" scale="0.001 0.001 0.001"/>
-    </geometry>
+    <!-- ここから SDF の surface/friction -->
+    <surface>
+      <friction>
+        <ode>
+          <mu>${wheel_surface_mu1}</mu>
+          <mu2>${wheel_surface_mu2}</mu2>
+        </ode>
+      </friction>
+      <contact>
+        <ode>
+          <kp>${wheel_kp}</kp>
+          <kd>${wheel_kd}</kd>
+          <minDepth>${wheel_minDepth}</minDepth>
+          <maxVel>${wheel_maxVel}</maxVel>
+        </ode>
+      </contact>
+    </surface>
   </collision>
 </link>
@@ -189,4 +271,21 @@
       <mesh filename="package://vehicle_4ws_description/meshes/new_wheel_3.stl" scale="0.001 0.001 0.001"/>
     </geometry>
+    <!-- ここから SDF の surface/friction -->
+    <surface>
+      <friction>
+        <ode>
+          <mu>${wheel_surface_mu1}</mu>
+          <mu2>${wheel_surface_mu2}</mu2>
+        </ode>
+      </friction>
+      <contact>
+        <ode>
+          <kp>${wheel_kp}</kp>
+          <kd>${wheel_kd}</kd>
+          <minDepth>${wheel_minDepth}</minDepth>
+          <maxVel>${wheel_maxVel}</maxVel>
+        </ode>
+      </contact>
+    </surface>
   </collision>
 </link>
@@ -209,44 +308,21 @@
       <mesh filename="package://vehicle_4ws_description/meshes/new_wheel_4.stl" scale="0.001 0.001 0.001"/>
     </geometry>
-  </collision>
-</link>
-<link name="new_hinge_2">
-  <inertial>
-    <origin xyz="-6.714468377322369e-05 2.540692444763515e-07 -0.1152300475191588" rpy="0 0 0"/>
-    <mass value="4.884144703315957"/>
-    <inertia ixx="0.039519" iyy="0.032652" izz="0.021551" ixy="0.0" iyz="0.0" ixz="-3e-05"/>
-  </inertial>
-  <visual>
-    <origin xyz="0.44955 0.34248 -0.356" rpy="0 0 0"/>
-    <geometry>
-      <mesh filename="package://vehicle_4ws_description/meshes/new_hinge_2.stl" scale="0.001 0.001 0.001"/>
-    </geometry>
-    <material name="_"/>
-  </visual>
-  <collision>
-    <origin xyz="0.44955 0.34248 -0.356" rpy="0 0 0"/>
-    <geometry>
-      <mesh filename="package://vehicle_4ws_description/meshes/new_hinge_2.stl" scale="0.001 0.001 0.001"/>
-    </geometry>
-  </collision>
-</link>
-<link name="new_hinge_4">
-  <inertial>
-    <origin xyz="-6.714468377405636e-05 2.5406924475390724e-07 -0.11523004751915963" rpy="0 0 0"/>
-    <mass value="4.884144703315957"/>
-    <inertia ixx="0.039519" iyy="0.032652" izz="0.021551" ixy="0.0" iyz="0.0" ixz="-3e-05"/>
-  </inertial>
-  <visual>
-    <origin xyz="0.44955 -0.45752 -0.356" rpy="0 0 0"/>
-    <geometry>
-      <mesh filename="package://vehicle_4ws_description/meshes/new_hinge_4.stl" scale="0.001 0.001 0.001"/>
-    </geometry>
-    <material name="_"/>
-  </visual>
-  <collision>
-    <origin xyz="0.44955 -0.45752 -0.356" rpy="0 0 0"/>
-    <geometry>
-      <mesh filename="package://vehicle_4ws_description/meshes/new_hinge_4.stl" scale="0.001 0.001 0.001"/>
-    </geometry>
+    <!-- ここから SDF の surface/friction -->
+    <surface>
+      <friction>
+        <ode>
+          <mu>${wheel_surface_mu1}</mu>
+          <mu2>${wheel_surface_mu2}</mu2>
+        </ode>
+      </friction>
+      <contact>
+        <ode>
+          <kp>${wheel_kp}</kp>
+          <kd>${wheel_kd}</kd>
+          <minDepth>${wheel_minDepth}</minDepth>
+          <maxVel>${wheel_maxVel}</maxVel>
+        </ode>
+      </contact>
+    </surface>
   </collision>
 </link>

Commit message: 摩擦修正

File: urdf/vehicle_4ws_real.xacro (robot description, xacro)
@@ -40,5 +40,5 @@
 <link name="body_link">
   <inertial>
-    <origin xyz="0.001411408730126027 0.05751189617802702 0.0" rpy="0 0 0"/>
+    <origin xyz="0.001411408730126027 0.05751189617802702 0.2" rpy="0 0 0"/>
     <mass value="${vehicle_body_mass}"/>
     <inertia ixx="${vehicle_inertia_coef*114.688091}" iyy="${vehicle_inertia_coef*336.418835}" izz="${vehicle_inertia_coef*418.647558}" ixy="${vehicle_inertia_coef*0.010139}" iyz="${vehicle_inertia_coef*0.002956}" ixz="${-vehicle_inertia_coef*0.33997}"/>

Commit message: 車輪のcollisionをcylinderに設定

File: urdf/vehicle_4ws_real.xacro (robot description, xacro)
@@ -193,7 +193,11 @@
   </visual>
   <collision>
-    <origin xyz="-0.450031 0.34248 -0.150215" rpy="0 0 0"/>
-    <geometry>
+    <!-- <origin xyz="-0.450031 0.34248 -0.150215" rpy="0 0 0"/> -->
+    <!-- <geometry>
       <mesh filename="package://vehicle_4ws_description/meshes/new_wheel_1.stl" scale="0.001 0.001 0.001"/>
+    </geometry> -->
+    <origin xyz="0 0 0" rpy="1.57 0 0"/>
+    <geometry>
+      <cylinder radius="0.16" length="0.05"/>
     </geometry>
     <!-- ここから SDF の surface/friction -->
@@ -230,7 +234,11 @@
   </visual>
   <collision>
-    <origin xyz="0.449969 0.34248 -0.150215" rpy="0 0 0"/>
+    <!-- <origin xyz="0.449969 0.34248 -0.150215" rpy="0 0 0"/>
     <geometry>
       <mesh filename="package://vehicle_4ws_description/meshes/new_wheel_2.stl" scale="0.001 0.001 0.001"/>
+    </geometry> -->
+    <origin xyz="0 0 0" rpy="1.57 0 0"/>
+    <geometry>
+      <cylinder radius="0.16" length="0.05"/>
     </geometry>
     <!-- ここから SDF の surface/friction -->
@@ -267,7 +275,11 @@
   </visual>
   <collision>
-    <origin xyz="-0.450031 -0.45752 -0.150215" rpy="0 0 0"/>
+    <!-- <origin xyz="-0.450031 -0.45752 -0.150215" rpy="0 0 0"/>
     <geometry>
       <mesh filename="package://vehicle_4ws_description/meshes/new_wheel_3.stl" scale="0.001 0.001 0.001"/>
+    </geometry> -->
+    <origin xyz="0 0 0" rpy="1.57 0 0"/>
+    <geometry>
+      <cylinder radius="0.16" length="0.05"/>
     </geometry>
     <!-- ここから SDF の surface/friction -->
@@ -304,7 +316,11 @@
   </visual>
   <collision>
-    <origin xyz="0.449969 -0.45752 -0.150215" rpy="0 0 0"/>
+    <!-- <origin xyz="0.449969 -0.45752 -0.150215" rpy="0 0 0"/>
     <geometry>
       <mesh filename="package://vehicle_4ws_description/meshes/new_wheel_4.stl" scale="0.001 0.001 0.001"/>
+    </geometry> -->
+    <origin xyz="0 0 0" rpy="1.57 0 0"/>
+    <geometry>
+      <cylinder radius="0.16" length="0.05"/>
     </geometry>
     <!-- ここから SDF の surface/friction -->
